File: kicad/controller.sch (KiCad schematic (older format))
At the start: 44 parts, among them J4 Handle, Q1 AO4407, Q2 BC847, Q3 BC857, Q4 BC847, U4 MCP602, U5 MCP602

Commit message: updated controller
Parts:
- R14: value 1k -> 1k1
- R16: value 150k -> 300k
Changed lines of the file:
@@
 P 3300 2500
 F 0 "R16" V 3400 2500 50  0000 C CNN
-F 1 "150k" V 3300 2500 50  0000 C CNN
+F 1 "300k" V 3300 2500 50  0000 C CNN
 F 2 "Resistor_SMD:R_0603_1608Metric" V 3230 2500 50  0001 C CNN
 F 3 "~" H 3300 2500 50  0001 C CNN
@@
 P 3000 2650
 F 0 "R14" H 2950 2650 50  0000 R CNN
-F 1 "1k" V 3000 2700 50  0000 R CNN
+F 1 "1k1" V 3000 2700 50  0000 R CNN
 F 2 "Resistor_SMD:R_0603_1608Metric" V 2930 2650 50  0001 C CNN
 F 3 "~" H 3000 2650 50  0001 C CNN

Commit message: Arlene v1.00
Parts:
- removed C18: 1u, Capacitor_SMD:C_0603_1608Metric, symbol Device:C
- removed C19, C20, C21, C22, C25, C26, C27, C28: nm, Capacitor_SMD:C_0603_1608Metric, symbol Device:C
- removed C24: 100n, Capacitor_SMD:C_0603_1608Metric, symbol Device:C
- removed D7: 1N4148, Diode_SMD:D_0805_2012Metric, symbol Device:D
- removed D8: 20v, Diode_SMD:D_0805_2012Metric, symbol Device:D_Zener
- removed Q2, Q4: BC847, Package_TO_SOT_SMD:SOT-23, symbol Transistor_BJT:BC847
- removed Q3: BC857, Package_TO_SOT_SMD:SOT-23, symbol Transistor_BJT:BC857
- removed R12: 56k, Resistor_SMD:R_0603_1608Metric, symbol Device:R
- removed R15: 100, Resistor_SMD:R_0603_1608Metric, symbol Device:R
- removed R17: 14k, Resistor_SMD:R_0603_1608Metric, symbol Device:R
- removed R18, R21, R30, R31: 470, Resistor_SMD:R_0603_1608Metric, symbol Device:R
- removed R26, R27: 10k, Resistor_SMD:R_0603_1608Metric, symbol Device:R
- removed unit 2 of U4
- removed unit 1 of U5
- removed unit 3 of U5
- added D2: 1N4148, Diode_SMD:D_SOD-323, symbol Device:D
- added Q2: AO3400A, Package_TO_SOT_SMD:SOT-23, symbol Device:Q_NMOS_GSD
- added R6: 100k, Resistor_SMD:R_0603_1608Metric, symbol Device:R
- J3: renamed from J4; footprint Connector_PinHeader_2.54mm:PinHeader_1x05_P2.54mm_Vertical -> Connector_JST:JST_XH_B5B-XH-A_1x05_P2.50mm_Vertical
- R12: renamed from R23; value 6k8 -> 10k
- R22: value 100 -> 10k
- R4: renamed from R19; value 5.1k -> 10k
- R5: renamed from R20; value 1k -> 2k
- R8: renamed from R35; value 4k7 -> 10k
- renumbered C23 to C14, R11 to R10, R25 to R11, R28 to R15, R24 to R16, R16 to R17, R29 to R18, R36 to R9, U5 to U4
Connections:
- net labels added: Earth, adc_handle_temperature, adc_heater_current, adc_heater_temperature, adc_heater_voltage, handle_switch_in, handle_temperature
- net labels removed: adc_current, adc_heater_temp, adc_thermistor_temp, adc_voltage, thermistor
- wire segments 60 -> 32
Other:
- note added: "0mV to 10mV"
- note removed: "0mV to 20mV"
- note removed: "10K ntc\n0C to 60C\n14.6uA to 200uA"
- note removed: "1V to 3.3V\n0C to 60C"
- moved on the sheet: C13, C14, J3, Q1, R10, R11, R12, R14, R15, R16, R17, R18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
