File: kicad/power.sch (KiCad schematic (older format))
At the start: 22 parts, among them J1 24v, U1 ACT4088, U2 LP5907-3.3

Commit message: Arlene v1.00
Parts:
- removed C2, C4, C7, C8: 100n, Capacitor_SMD:C_0603_1608Metric, symbol Device:C
- removed C6: nm, Capacitor_SMD:C_0603_1608Metric, symbol Device:C
- removed C9: 10u, Capacitor_SMD:C_0805_2012Metric, symbol Device:C
- removed D1, D2: D_Schottky, Diode_SMD:D_0805_2012Metric, symbol Device:D_Schottky
- removed J1: 24v, Connector_BarrelJack:BarrelJack_Horizontal, symbol Connector:Barrel_Jack_Switch
- removed L2: Ferrite, Inductor_SMD:L_0805_2012Metric, symbol Device:L_Core_Ferrite_Small
- removed U2: LP5907-3.3, Package_TO_SOT_SMD:SOT-23-5, symbol arlene:LP5907-3.3-2-0
- added C17: 100u, Capacitor_Tantalum_SMD:CP_EIA-7343-31_Kemet-D, symbol Device:CP
- added J4: Power, Connector_JST:JST_XH_B3B-XH-A_1x03_P2.50mm_Vertical, symbol Connector_Generic:Conn_01x03
- added U2: XC6206PxxxMR, Package_TO_SOT_SMD:SOT-23, symbol Regulator_Linear:XC6206PxxxMR
- L1: footprint arlene:L_4x4_H1.75 -> arlene:L_4.1x4.1_H1.75
- renumbered C5 to C2, C30 to C4, C10 to C5, C29 to C6, D4 to D1, R4 to R1, R5 to R2
Connections:
- net labels added: +5V, Earth
- net labels removed: switch_5v, usb_vbus
- wire segments 29 -> 27
Other:
- moved on the sheet: C1, C2, C3, C4, C5, C6, D1, L1, R1, R2, U1
