File: kicad/processor.sch (KiCad schematic (older format))
At the start: 31 parts, among them J2 Display, J3 Debug, J5 USB-C, J6 Remote, SW1 Encoder, U3 STM32F072C8Tx, U6 SRV05-4

Commit message: Arlene v1.00
Parts:
- removed D3, D6: LED_CRGB, LED_THT:LED_D5.0mm-4_RGB, symbol Device:LED_CRGB
- removed H1, H2, H3, H4: MountingHole, MountingHole:MountingHole_2.5mm, symbol Mechanical:MountingHole
- removed J2: Display, Connector_PinHeader_2.54mm:PinHeader_1x04_P2.54mm_Vertical, symbol Connector_Generic:Conn_01x04
- removed J3: Debug, Connector_PinHeader_2.54mm:PinHeader_2x04_P2.54mm_Vertical, symbol Connector_Generic:Conn_02x04_Odd_Even
- removed J6: Remote, Connector_PinSocket_2.54mm:PinSocket_2x04_P2.54mm_Vertical, symbol Connector_Generic:Conn_02x04_Odd_Even
- removed R1, R2: 5k1, Resistor_SMD:R_0603_1608Metric, symbol Device:R
- removed R3, R32, R33, R34, R8, R9: R, Resistor_SMD:R_0603_1608Metric, symbol Device:R
- removed R6: 4k7, Resistor_SMD:R_0603_1608Metric, symbol Device:R
- removed U6: SRV05-4, Package_TO_SOT_SMD:SOT-23-6, symbol Power_Protection:SRV05-4
- added C11, C15: 1n, Capacitor_SMD:C_0603_1608Metric, symbol Device:C
- added D3: LED_RCGB, arlene:LED_D5.0mm-4_RGB, symbol Device:LED_RCGB
- added J1: Display, Connector_PinHeader_2.54mm:PinHeader_1x07_P2.54mm_Vertical, symbol Connector_Generic:Conn_01x07
- added J2: Debug, Connector_PinHeader_2.54mm:PinHeader_2x04_P2.54mm_Vertical, symbol Connector_Generic:Conn_02x04_Odd_Even
- added R19, R20, R21: 1k, Resistor_SMD:R_0603_1608Metric, symbol Device:R
- added R23, R24: 4k7, Resistor_SMD:R_0603_1608Metric, symbol Device:R
- added R25: 100, Resistor_SMD:R_0603_1608Metric, symbol Device:R
- C16: value 100n -> 1n
- J5: footprint Connector_USB:USB_C_Receptacle_XKB_U262-16XN-4BVC11 -> arlene:usb-c_14pin_tht_vertical
- SW1: footprint Rotary_Encoder:RotaryEncoder_Alps_EC12E-Switch_Vertical_H20mm -> arlene:RotaryEncoder_Alps_EC12E-Switch_Vertical_H20mm
- renumbered C15 to C10, C17 to C12, C12 to C7, C11 to C8, C14 to C9, R10 to R3
Connections:
- net labels added: +5V, adc_handle_temperature, adc_heater_current, adc_heater_temperature, adc_heater_voltage, handle_switch_in, led_blue, led_green, led_red, oled_cs, oled_dc, oled_reset, oled_sck, oled_sda
- net labels removed: adc_current, adc_heater_temp, adc_thermistor_temp, adc_voltage, handle_switch, i2c_scl, i2c_sda, led1_blue, led1_green, led1_red, led2_blue, led2_green, led2_red, usb_vbus
- wire segments 25 -> 34
- no-connect marks 15 -> 16
Other:
- moved on the sheet: BZ1, C10, C12, C7, C8, C9, R3, SW1
